Commit message: dodano symulowanie sensorow ahrs, dvl i cisnienia - sim driver i urdf; przerzucono wszystkie sim drivery do bringup

File: src/bluerov2_description/urdf/bluerov2.xacro (robot description, xacro)
@@ -38,3 +38,27 @@
   </link>
   <xacro:include filename="thrusters.xacro"/>
+  <!-- Sensor frames — czyste ramki TF, bez pluginów symulacyjnych.
+       Szum i model sensoryczny w sim_sensor_drivers.py (robot_bringup).
+       Na HW te pozycje wyznaczają lever arm dla EKF. -->
+  <!-- AHRS (MTi-600): wewnątrz rury elektronicznej, środek-góra kadłuba -->
+  <link name="${ns}/ahrs_link"/>
+  <joint name="${ns}/ahrs_joint" type="fixed">
+    <parent link="${ns}/base_link"/>
+    <child  link="${ns}/ahrs_link"/>
+    <origin xyz="0.0 0.0 0.06" rpy="0 0 0"/>
+  </joint>
+  <!-- DVL: spód kadłuba, lekko z tyłu; Z obrócone o PI — wskazuje w dół (w stronę dna) -->
+  <link name="${ns}/dvl_link"/>
+  <joint name="${ns}/dvl_joint" type="fixed">
+    <parent link="${ns}/base_link"/>
+    <child  link="${ns}/dvl_link"/>
+    <origin xyz="-0.05 0.0 -0.12" rpy="${pi} 0 0"/>
+  </joint>
+  <!-- Depth (Bar30): bok ramy, wystawiony na wodę -->
+  <link name="${ns}/depth_link"/>
+  <joint name="${ns}/depth_joint" type="fixed">
+    <parent link="${ns}/base_link"/>
+    <child  link="${ns}/depth_link"/>
+    <origin xyz="0.0 0.15 0.0" rpy="0 0 0"/>
+  </joint>
 </robot>

Commit message: dodanie symbolicznej masy czujnikow; dostrojenie pid i ekf; rozdzielenie parametrow sim i z rosa; dodanie marchewki do plannera by regulowac pozycje setpoint; nowe tryby CRUISE i WORK

File: src/bluerov2_description/urdf/bluerov2.xacro (robot description, xacro)
@@ -42,5 +42,7 @@
        Na HW te pozycje wyznaczają lever arm dla EKF. -->
   <!-- AHRS (MTi-600): wewnątrz rury elektronicznej, środek-góra kadłuba -->
-  <link name="${ns}/ahrs_link"/>
+  <link name="${ns}/ahrs_link">
+    <inertial><mass value="0.001"/><inertia ixx="1e-6" iyy="1e-6" izz="1e-6" ixy="0" ixz="0" iyz="0"/></inertial>
+  </link>
   <joint name="${ns}/ahrs_joint" type="fixed">
     <parent link="${ns}/base_link"/>
@@ -49,5 +51,7 @@
   </joint>
   <!-- DVL: spód kadłuba, lekko z tyłu; Z obrócone o PI — wskazuje w dół (w stronę dna) -->
-  <link name="${ns}/dvl_link"/>
+  <link name="${ns}/dvl_link">
+    <inertial><mass value="0.001"/><inertia ixx="1e-6" iyy="1e-6" izz="1e-6" ixy="0" ixz="0" iyz="0"/></inertial>
+  </link>
   <joint name="${ns}/dvl_joint" type="fixed">
     <parent link="${ns}/base_link"/>
@@ -56,5 +60,7 @@
   </joint>
   <!-- Depth (Bar30): bok ramy, wystawiony na wodę -->
-  <link name="${ns}/depth_link"/>
+  <link name="${ns}/depth_link">
+    <inertial><mass value="0.001"/><inertia ixx="1e-6" iyy="1e-6" izz="1e-6" ixy="0" ixz="0" iyz="0"/></inertial>
+  </link>
   <joint name="${ns}/depth_joint" type="fixed">
     <parent link="${ns}/base_link"/>
